File: multipreamp-1.brd (EAGLE design)
At the start: 100 x 80 mm, 8 parts

Commit message: Desenvolvimento do esquematico
Parts:
- added C10, C12, C13, C15, C16, C17, C22, C23, C33, C9: (no value), rcl:C025-025X050
- added C11, C14, C18, C19, C20, C21, C24, C25, C4, C5, C6, C7, C8: (no value), rcl:C050-025X075
- added C26, C27, C29, C30, C31, C32: (no value), rcl:E2,5-6
- added C28: 100n SMD, rcl:C0805
- added D1, D2, D3, D4, D5, D6: 1N4148, diode:DO35-7
- added JP1, JP10, JP11, JP12, JP13, JP14, JP2, JP3, JP4, JP5, JP6, JP7, JP8, JP9: (no value), pinhead:1X01
- added POT_BASS, POT_GAIN, POT_MIDS, POT_TONE/TREBLE, POT_VOL: (no value), gm-pots:16MM-PCB-MOUNT
- added Q1, Q2, Q3, Q4, Q6, Q7: J201, gm-trans:TO92-
- added Q5: 2N5088, gm-trans:TO92-
- added R10, R11, R13, R14, R15, R16, R19, R20, R21, R22, R25, R26, R27, R28, R30, R31, R32, R33, R34, R35, R36, R37, R38, R39, R4, R5, R7, R8, R9: (no value), rcl:0207/7
- added R12, R18, R24, R40, R41: 1M SMD, rcl:R0805
- added R17, R23, R29, R6: (no value), rcl:RTRIM64W
- added R42, R43: 10k SMD, rcl:R0805
- added SJ1: (no value), jumper:SJ
- moved LED1 119.8 mm to (96.5, 24.1), turned to 90 degrees
- moved R3 113.1 mm to (82.5, 15.2), turned to 90 degrees
- moved LED2 111.2 mm to (88.9, 24.1), turned to 90 degrees
- moved C3 104.3 mm to (82.5, 24.1), turned to 90 degrees
- moved C1 101.6 mm to (77.5, 21.6), turned to 90 degrees
- moved R2 100.8 mm to (72.4, 17.8), turned to 90 degrees
- moved C2 94.2 mm to (77.5, 29.2), turned to 90 degrees
- moved R1 90.2 mm to (72.4, 27.9), turned to 90 degrees
Connections:
- new net N$1: C4.2, JP4.1, R5.2
- new net N$10: C26.+, Q6.1, R40.1
- new net N$11: C33.2, POT_GAIN.3, POT_TONE/TREBLE.2
- new net N$12: POT_GAIN.1, R11.2
- new net N$13: C33.1, C8.1, R12.2, R13.2, R14.2
- new net N$15: C11.2, C27.-, JP1.1, Q2.3, Q7.2, R17.2, R17.3
- new net N$16: C30.+, Q2.2, R15.2
- new net N$17: R15.1, R16.2
- new net N$18: C11.1, R18.2, R19.2, R20.2
- new net N$19: C12.2, C13.2, D3.C, D4.A, Q3.1, R20.1
- new net N$2: C4.1, Q1.2, R4.2
- new net N$20: C31.+, Q3.2, R21.2
- new net N$21: R21.1, R22.2
- new net N$22: C14.2, Q3.3, R23.2, R23.3
- new net N$23: C18.1, R30.1, R31.2, R32.1
- new net N$24: C14.1, R24.2, R25.2, R26.2
- new net N$25: C15.2, C16.2, D5.C, D6.A, Q4.1, R26.1
- new net N$26: C32.+, Q4.2, R27.2
- new net N$27: R27.1, R28.2
- new net N$28: JP2.1, Q4.3, R29.2, R29.3
- new net N$29: JP3.1, R30.2
- new net N$3: C8.2, POT_GAIN.2
- new net N$30: C17.2, Q5.2, R32.2
- new net N$31: C18.2, C19.1, Q5.3, R33.1
- new net N$32: C19.2, C20.1, R34.1, R35.1
- new net N$33: C21.2, R35.2, R36.1
- new net N$34: C20.2, POT_VOL.3, R36.2, R37.2
- new net N$35: JP10.1, POT_VOL.2
- new net N$37: C25.1, POT_MIDS.3, SJ1.1
- new net N$39: C24.2, C25.2, R38.2
- new net N$4: C1.2, LED1.A, LED2.K, Q1.1, R1.2
- new net N$40: C27.+, Q7.1, R41.1
- new net N$41: C22.1, C23.1, R38.1
- new net N$42: C10.2, C9.2, D1.C, D2.A, Q2.1, R14.1
- new net N$43: POT_BASS.1, R39.1, SJ1.2
- new net N$5: JP8.1, R1.1, R2.2, R3.2
- new net N$6: C7.2, JP6.1, R9.2
- new net N$7: C2.1, C5.2, R8.1
- new net N$8: C2.2, C26.-, Q1.3, Q6.2, R6.2, R6.3
- new net N$9: C6.1, C7.1, R10.1, R8.2
- new net TONE/TREBLE_1: C24.1, POT_BASS.2, POT_BASS.3, POT_TONE/TREBLE.1, R10.2
- new net TONE/TREBLE_3: C22.2, C23.2, C5.1, POT_TONE/TREBLE.3, R7.1
- new net V+: Q5.1, Q6.3, Q7.3, R17.1, R23.1, R29.1, R31.1, R42.1, R6.1
- new net VCC/2: C28.1, C29.+, R40.2, R41.2, R42.2, R43.1
- net GND: now also C1.1, C10.1, C12.1, C13.1, C15.1, C16.1, C17.1, C21.1, C28.2, C29.-, C30.-, C31.-, C32.-, C6.2, C9.1, D1.A, D2.C, D3.A, D4.C, D5.A, D6.C, JP11.1, JP12.1, JP13.1, JP14.1, JP5.1, JP7.1, JP9.1, LED1.K, LED2.A, POT_MIDS.1, POT_MIDS.2, POT_VOL.1, R11.1, R12.1, R13.1, R16.1, R18.1, R19.1, R22.1, R24.1, R25.1, R28.1, R3.1, R33.2, R34.2, R37.1, R39.2, R4.1, R43.2, R5.1, R7.2, R9.1
Other:
- board size 100 x 80 mm -> 100 x 50 mm

Commit message: Desenvolvimento do esquematico
Parts:
- added SJ2: (no value), jumper:SJ
- added TP1, TP2: PTR1PAD1-13, testpad:P1-13
- moved POT_VOL 2.54 mm to (90.2, 45.7)
- moved POT_GAIN 2.54 mm to (8.89, 45.7)
- moved POT_TONE/TREBLE 1.27 mm to (29.2, 45.7)
- moved POT_BASS 1.27 mm to (69.8, 45.7)
Connections:
- net N$22: now also TP2.TP
- net N$28: now also SJ2.1
- net N$29: now also SJ2.2
- net N$8: now also TP1.TP
Changed lines of the file:
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@@
 <element name="R9" library="rcl" package="0207/7" value="" x="87.63" y="8.89" rot="R90"/>
 <element name="R10" library="rcl" package="0207/7" value="" x="92.71" y="8.89" rot="R90"/>
-<element name="POT_TONE/TREBLE" library="gm-pots" package="16MM-PCB-MOUNT" value="" x="30.48" y="45.72"/>
-<element name="POT_GAIN" library="gm-pots" package="16MM-PCB-MOUNT" value="" x="11.43" y="45.72"/>
+<element name="POT_TONE/TREBLE" library="gm-pots" package="16MM-PCB-MOUNT" value="" x="29.21" y="45.72"/>
+<element name="POT_GAIN" library="gm-pots" package="16MM-PCB-MOUNT" value="" x="8.89" y="45.72"/>
 <element name="R11" library="rcl" package="0207/7" value="" x="-74.93" y="-60.96"/>
 <element name="C8" library="rcl" package="C050-025X075" value="" x="-74.93" y="-66.04"/>
@@
 <element name="C20" library="rcl" package="C050-025X075" value="" x="-95.25" y="-303.53"/>
 <element name="C21" library="rcl" package="C050-025X075" value="" x="-95.25" y="-308.61"/>
-<element name="POT_VOL" library="gm-pots" package="16MM-PCB-MOUNT" value="" x="87.63" y="45.72"/>
+<element name="POT_VOL" library="gm-pots" package="16MM-PCB-MOUNT" value="" x="90.17" y="45.72"/>
 <element name="JP4" library="pinhead" package="1X01" value="" x="-115.57" y="-313.69"/>
 <element name="JP5" library="pinhead" package="1X01" value="" x="-115.57" y="-318.77"/>
@@
 <element name="JP10" library="pinhead" package="1X01" value="" x="-115.57" y="-349.25"/>
 <element name="JP11" library="pinhead" package="1X01" value="" x="-115.57" y="-354.33"/>
-<element name="POT_BASS" library="gm-pots" package="16MM-PCB-MOUNT" value="" x="68.58" y="45.72"/>
+<element name="POT_BASS" library="gm-pots" package="16MM-PCB-MOUNT" value="" x="69.85" y="45.72"/>
 <element name="POT_MIDS" library="gm-pots" package="16MM-PCB-MOUNT" value="" x="49.53" y="45.72"/>
 <element name="C22" library="rcl" package="C025-025X050" value="" x="-171.45" y="-359.41"/>
@@
 <element name="C32" library="rcl" package="E2,5-6" value="" x="-171.45" y="-494.03"/>
 <element name="C33" library="rcl" package="C025-025X050" value="" x="-171.45" y="-500.38"/>
+<element name="TP1" library="testpad" package="P1-13" value="PTR1PAD1-13" x="-172.72" y="-505.46">
+<attribute name="TP_SIGNAL_NAME" value="" x="-172.72" y="-505.46" size="1.778" layer="27" display="off"/>
+</element>
+<element name="TP2" library="testpad" package="P1-13" value="PTR1PAD1-13" x="-172.72" y="-510.54">
+<attribute name="TP_SIGNAL_NAME" value="" x="-172.72" y="-510.54" size="1.778" layer="27" display="off"/>
+</element>
+<element name="SJ2" library="jumper" package="SJ" value="" x="-172.72" y="-515.62"/>
 </elements>
 <signals>
@@
 <wire x1="88.9" y1="22.86" x2="82.55" y2="14.29" width="0" layer="19" extent="1-1"/>
 <wire x1="96.52" y1="25.4" x2="88.9" y2="22.86" width="0" layer="19" extent="1-1"/>
-<wire x1="92.71" y1="45.72" x2="96.52" y2="25.4" width="0" layer="19" extent="1-1"/>
+<wire x1="95.25" y1="45.72" x2="96.52" y2="25.4" width="0" layer="19" extent="1-1"/>
 <wire x1="54.61" y1="45.72" x2="57.15" y2="13.97" width="0" layer="19" extent="1-1"/>
 <wire x1="49.53" y1="45.72" x2="54.61" y2="45.72" width="0" layer="19" extent="1-1"/>
@@
 <contactref element="POT_GAIN" pad="3"/>
 <contactref element="C33" pad="2"/>
-<wire x1="6.35" y1="45.72" x2="-170.18" y2="-500.38" width="0" layer="19" extent="1-1"/>
-<wire x1="30.48" y1="45.72" x2="6.35" y2="45.72" width="0" layer="19" extent="1-1"/>
+<wire x1="3.81" y1="45.72" x2="-170.18" y2="-500.38" width="0" layer="19" extent="1-1"/>
+<wire x1="29.21" y1="45.72" x2="3.81" y2="45.72" width="0" layer="19" extent="1-1"/>
 </signal>
 <signal name="N$12">
 <contactref element="POT_GAIN" pad="1"/>
 <contactref element="R11" pad="2"/>
-<wire x1="16.51" y1="45.72" x2="-71.12" y2="-60.96" width="0" layer="19" extent="1-1"/>
+<wire x1="13.97" y1="45.72" x2="-71.12" y2="-60.96" width="0" layer="19" extent="1-1"/>
 </signal>
 <signal name="N$3">
 <contactref element="POT_GAIN" pad="2"/>
 <contactref element="C8" pad="2"/>
-<wire x1="11.43" y1="45.72" x2="-72.39" y2="-66.04" width="0" layer="19" extent="1-1"/>
+<wire x1="8.89" y1="45.72" x2="-72.39" y2="-66.04" width="0" layer="19" extent="1-1"/>
 </signal>
 <signal name="N$13">
@@
 <contactref element="C14" pad="2"/>
 <contactref element="R23" pad="2"/>
+<contactref element="TP2" pad="TP"/>
+<wire x1="-78.74" y1="-214.63" x2="-172.72" y2="-510.54" width="0" layer="19" extent="1-1"/>
 <wire x1="-93.98" y1="-186.69" x2="-78.74" y2="-214.63" width="0" layer="19" extent="1-1"/>
 <wire x1="-93.98" y1="-184.15" x2="-93.98" y2="-186.69" width="0" layer="19" extent="1-1"/>
@@
 <contactref element="JP2" pad="1"/>
 <contactref element="R29" pad="2"/>
+<contactref element="SJ2" pad="1"/>
+<wire x1="-96.52" y1="-234.95" x2="-173.482" y2="-515.62" width="0" layer="19" extent="1-1"/>
 <wire x1="-93.98" y1="-198.12" x2="-96.52" y2="-234.95" width="0" layer="19" extent="1-1"/>
 <wire x1="-93.98" y1="-195.58" x2="-93.98" y2="-198.12" width="0" layer="19" extent="1-1"/>
@@
 <contactref element="R30" pad="2"/>
 <contactref element="JP3" pad="1"/>
-<wire x1="-90.17" y1="-245.11" x2="-96.52" y2="-240.03" width="0" layer="19" extent="1-1"/>
+<contactref element="SJ2" pad="2"/>
+<wire x1="-90.17" y1="-245.11" x2="-171.958" y2="-515.62" width="0" layer="19" extent="1-1"/>
+<wire x1="-96.52" y1="-240.03" x2="-90.17" y2="-245.11" width="0" layer="19" extent="1-1"/>
 </signal>
 <signal name="N$30">
@@
 <contactref element="POT_VOL" pad="3"/>
 <contactref element="R37" pad="2"/>
-<wire x1="82.55" y1="45.72" x2="-109.22" y2="-334.01" width="0" layer="19" extent="1-1"/>
-<wire x1="-92.71" y1="-303.53" x2="82.55" y2="45.72" width="0" layer="19" extent="1-1"/>
+<wire x1="85.09" y1="45.72" x2="-109.22" y2="-334.01" width="0" layer="19" extent="1-1"/>
+<wire x1="-92.71" y1="-303.53" x2="85.09" y2="45.72" width="0" layer="19" extent="1-1"/>
 <wire x1="-90.17" y1="-298.45" x2="-92.71" y2="-303.53" width="0" layer="19" extent="1-1"/>
 </signal>
@@
 <contactref element="POT_VOL" pad="2"/>
 <contactref element="JP10" pad="1"/>
-<wire x1="87.63" y1="45.72" x2="-115.57" y2="-349.25" width="0" layer="19" extent="1-1"/>
+<wire x1="90.17" y1="45.72" x2="-115.57" y2="-349.25" width="0" layer="19" extent="1-1"/>
 </signal>
 <signal name="TONE/TREBLE_1">
@@
 <contactref element="R10" pad="2"/>
 <contactref element="POT_TONE/TREBLE" pad="1"/>
-<wire x1="68.58" y1="45.72" x2="63.5" y2="45.72" width="0" layer="19" extent="1-1"/>
-<wire x1="-172.72" y1="-389.89" x2="63.5" y2="45.72" width="0" layer="19" extent="1-1"/>
-<wire x1="92.71" y1="12.7" x2="68.58" y2="45.72" width="0" layer="19" extent="1-1"/>
-<wire x1="35.56" y1="45.72" x2="92.71" y2="12.7" width="0" layer="19" extent="1-1"/>
+<wire x1="69.85" y1="45.72" x2="64.77" y2="45.72" width="0" layer="19" extent="1-1"/>
+<wire x1="-172.72" y1="-389.89" x2="64.77" y2="45.72" width="0" layer="19" extent="1-1"/>
+<wire x1="92.71" y1="12.7" x2="69.85" y2="45.72" width="0" layer="19" extent="1-1"/>
+<wire x1="34.29" y1="45.72" x2="92.71" y2="12.7" width="0" layer="19" extent="1-1"/>
 </signal>
 <signal name="N$37">
@@
 <contactref element="R7" pad="1"/>
 <contactref element="POT_TONE/TREBLE" pad="3"/>
-<wire x1="72.39" y1="5.08" x2="25.4" y2="45.72" width="0" layer="19" extent="1-1"/>
+<wire x1="72.39" y1="5.08" x2="24.13" y2="45.72" width="0" layer="19" extent="1-1"/>
 <wire x1="62.23" y1="5.08" x2="72.39" y2="5.08" width="0" layer="19" extent="1-1"/>
-<wire x1="-170.18" y1="-359.41" x2="25.4" y2="45.72" width="0" layer="19" extent="1-1"/>
+<wire x1="-170.18" y1="-359.41" x2="24.13" y2="45.72" width="0" layer="19" extent="1-1"/>
 <wire x1="-170.18" y1="-364.49" x2="-170.18" y2="-359.41" width="0" layer="19" extent="1-1"/>
 </signal>
@@
 <contactref element="R39" pad="1"/>
 <contactref element="SJ1" pad="2"/>
-<wire x1="-173.99" y1="-384.81" x2="73.66" y2="45.72" width="0" layer="19" extent="1-1"/>
+<wire x1="-173.99" y1="-384.81" x2="74.93" y2="45.72" width="0" layer="19" extent="1-1"/>
 <wire x1="-171.958" y1="-394.97" x2="-173.99" y2="-384.81" width="0" layer="19" extent="1-1"/>
 </signal>
@@
 <contactref element="C2" pad="2"/>
 <contactref element="C26" pad="-"/>
-<wire x1="52.07" y1="8.89" x2="77.47" y2="31.75" width="0" layer="19" extent="1-1"/>
-<wire x1="49.53" y1="8.89" x2="52.07" y2="8.89" width="0" layer="19" extent="1-1"/>
-<wire x1="39.37" y1="13.97" x2="49.53" y2="8.89" width="0" layer="19" extent="1-1"/>
-<wire x1="-171.45" y1="-398.78" x2="39.37" y2="13.97" width="0" layer="19" extent="1-1"/>
-<wire x1="-170.18" y1="-406.4" x2="-171.45" y2="-398.78" width="0" layer="19" extent="1-1"/>
+<contactref element="TP1" pad="TP"/>
+<wire x1="-170.18" y1="-406.4" x2="-172.72" y2="-505.46" width="0" layer="19" extent="1-1"/>
+<wire x1="-171.45" y1="-398.78" x2="-170.18" y2="-406.4" width="0" layer="19" extent="1-1"/>
+<wire x1="39.37" y1="13.97" x2="-171.45" y2="-398.78" width="0" layer="19" extent="1-1"/>
+<wire x1="49.53" y1="8.89" x2="39.37" y2="13.97" width="0" layer="19" extent="1-1"/>
+<wire x1="52.07" y1="8.89" x2="49.53" y2="8.89" width="0" layer="19" extent="1-1"/>
+<wire x1="77.47" y1="31.75" x2="52.07" y2="8.89" width="0" layer="19" extent="1-1"/>
 </signal>
 <signal name="N$10">

Commit message: Desenvolvimento do esquematico
Parts:
- removed JP8: (no value), pinhead:1X01
- added JP_IN: (no value), pinhead:1X01
- LED1, LED2: device led:LED5MM -> led:LED3MM
- R2: device rcl:0207/7 -> rcl:0207/5V
- moved JP9 367.5 mm to (6.35, 2.54)
- moved LED1 91.6 mm to (5.08, 29.2), turned to 180 degrees
- moved LED2 83.8 mm to (5.08, 24.1), turned to 0 degrees
- moved R3 77.6 mm to (5.08, 10.2), turned to 0 degrees
- moved C1 73.8 mm to (3.81, 16.5)
- moved R2 67.7 mm to (5.08, 10.2), turned to 0 degrees
- moved R1 65.8 mm to (7.62, 16.5)
- moved R6 42.6 mm to (14.0, 26.7)
- moved Q1 28.2 mm to (11.4, 20.3), turned to 270 degrees
- renumbered JP10 to JP_OUT
Connections:
- net N$5: now also JP_IN.1; no longer JP8.1
