File: multipreamp-1.sch (EAGLE design)
At the start: 8 parts

Commit message: Desenvolvimento do esquematico
Parts:
- added C10, C12, C13, C15, C16, C17, C22, C23, C33, C9: (no value), rcl:C-EU025-025X050
- added C11, C14, C18, C19, C20, C21, C24, C25, C4, C5, C6, C7, C8: (no value), rcl:C-EU050-025X075
- added C26, C27, C29, C30, C31, C32: (no value), rcl:CPOL-EUE2.5-6
- added C28: 100n SMD, rcl:C-EUC0805
- added D1, D2, D3, D4, D5, D6: 1N4148, diode:1N4148DO35-7
- added JP1, JP10, JP11, JP12, JP13, JP14, JP2, JP3, JP4, JP5, JP6, JP7, JP8, JP9: (no value), pinhead:PINHD-1X1
- added POT_BASS, POT_GAIN, POT_MIDS, POT_TONE/TREBLE, POT_VOL: (no value), gm-pots:POTPCB
- added Q1, Q2, Q3, Q4, Q6, Q7: J201, gm-trans:J201
- added Q5: 2N5088, gm-trans:2N5088
- added R10, R11, R13, R14, R15, R16, R19, R20, R21, R22, R25, R26, R27, R28, R30, R31, R32, R33, R34, R35, R36, R37, R38, R39, R4, R5, R7, R8, R9: (no value), rcl:R-US_0207/7
- added R12, R18, R24, R40, R41: 1M SMD, rcl:R-US_R0805
- added R17, R23, R29, R6: (no value), rcl:R-TRIMM64W
- added R42, R43: 10k SMD, rcl:R-US_R0805
- added SJ1: (no value), jumper:SJ
Connections:
- new net N$1: C4.2, JP4.1, R5.2
- new net N$10: C26.+, Q6.G, R40.1
- new net N$11: C33.2, POT_GAIN.3, POT_TONE/TREBLE.2
- new net N$12: POT_GAIN.1, R11.2
- new net N$13: C33.1, C8.1, R12.2, R13.2, R14.2
- new net N$15: C11.2, C27.-, JP1.1, Q2.D, Q7.S, R17.E, R17.S
- new net N$16: C30.+, Q2.S, R15.2
- new net N$17: R15.1, R16.2
- new net N$18: C11.1, R18.2, R19.2, R20.2
- new net N$19: C12.2, C13.2, D3.C, D4.A, Q3.G, R20.1
- new net N$2: C4.1, Q1.S, R4.2
- new net N$20: C31.+, Q3.S, R21.2
- new net N$21: R21.1, R22.2
- new net N$22: C14.2, Q3.D, R23.E, R23.S
- new net N$23: C18.1, R30.1, R31.2, R32.1
- new net N$24: C14.1, R24.2, R25.2, R26.2
- new net N$25: C15.2, C16.2, D5.C, D6.A, Q4.G, R26.1
- new net N$26: C32.+, Q4.S, R27.2
- new net N$27: R27.1, R28.2
- new net N$28: JP2.1, Q4.D, R29.E, R29.S
- new net N$29: JP3.1, R30.2
- new net N$3: C8.2, POT_GAIN.2
- new net N$30: C17.2, Q5.B, R32.2
- new net N$31: C18.2, C19.1, Q5.E, R33.1
- new net N$32: C19.2, C20.1, R34.1, R35.1
- new net N$33: C21.2, R35.2, R36.1
- new net N$34: C20.2, POT_VOL.3, R36.2, R37.2
- new net N$35: JP10.1, POT_VOL.2
- new net N$37: C25.1, POT_MIDS.3, SJ1.1
- new net N$39: C24.2, C25.2, R38.2
- new net N$4: C1.2, LED1.A, LED2.C, Q1.G, R1.2
- new net N$40: C27.+, Q7.G, R41.1
- new net N$41: C22.1, C23.1, R38.1
- new net N$42: C10.2, C9.2, D1.C, D2.A, Q2.G, R14.1
- new net N$43: POT_BASS.1, R39.1, SJ1.2
- new net N$5: JP8.1, R1.1, R2.2, R3.2
- new net N$6: C7.2, JP6.1, R9.2
- new net N$7: C2.1, C5.2, R8.1
- new net N$8: C2.2, C26.-, Q1.D, Q6.S, R6.E, R6.S
- new net N$9: C6.1, C7.1, R10.1, R8.2
- new net TONE/TREBLE_1: C24.1, POT_BASS.2, POT_BASS.3, POT_TONE/TREBLE.1, R10.2
- new net TONE/TREBLE_3: C22.2, C23.2, C5.1, POT_TONE/TREBLE.3, R7.1
- new net V+: Q5.C, Q6.D, Q7.D, R17.A, R23.A, R29.A, R31.1, R42.1, R6.A
- new net VCC/2: C28.1, C29.+, R40.2, R41.2, R42.2, R43.1
- net GND: now also C1.1, C10.1, C12.1, C13.1, C15.1, C16.1, C17.1, C21.1, C28.2, C29.-, C30.-, C31.-, C32.-, C6.2, C9.1, D1.A, D2.C, D3.A, D4.C, D5.A, D6.C, JP11.1, JP12.1, JP13.1, JP14.1, JP5.1, JP7.1, JP9.1, LED1.C, LED2.A, POT_MIDS.1, POT_MIDS.2, POT_VOL.1, R11.1, R12.1, R13.1, R16.1, R18.1, R19.1, R22.1, R24.1, R25.1, R28.1, R3.1, R33.2, R34.2, R37.1, R39.2, R4.1, R43.2, R5.1, R7.2, R9.1
Other:
- note added: "AZABACHE BRIGHT"
- note added: "AZABACHE SCOOP"
- note added: "Fender - montar jumper e deixar R39 em aberto"
- note added: "Umble - montar R39 e deixar jumper em aberto"
- moved on the sheet: C3

Commit message: Desenvolvimento do esquematico
Parts:
- added SJ2: (no value), jumper:SJ
- added TP1, TP2: PTR1PAD1-13, testpad:PTR1PAD1-13
Connections:
- net N$22: now also TP2.TP
- net N$28: now also SJ2.1
- net N$29: now also SJ2.2
- net N$8: now also TP1.TP
Other:
- moved on the sheet: C17, C18, C19, C20, C21, JP10, JP11, JP14, JP3, POT_VOL, Q5, R23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

Commit message: Desenvolvimento do esquematico
Parts:
- LED1, LED2: device led:LED5MM -> led:LED3MM
- R2: device rcl:R-US_0207/7 -> rcl:R-US_0207/5V
- renumbered JP10 to JP_OUT, JP8 to JP_IN
Changed lines of the file:
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@@
 <grid distance="0.1" unitdist="inch" unit="inch" style="lines" multiple="1" display="no" altdistance="0.01" altunitdist="inch" altunit="inch"/>
 <layers>
-<layer number="1" name="Top" color="4" fill="1" visible="no" active="no"/>
-<layer number="16" name="Bottom" color="1" fill="1" visible="no" active="no"/>
-<layer number="17" name="Pads" color="2" fill="1" visible="no" active="no"/>
-<layer number="18" name="Vias" color="2" fill="1" visible="no" active="no"/>
-<layer number="19" name="Unrouted" color="6" fill="1" visible="no" active="no"/>
-<layer number="20" name="Dimension" color="15" fill="1" visible="no" active="no"/>
-<layer number="21" name="tPlace" color="7" fill="1" visible="no" active="no"/>
-<layer number="22" name="bPlace" color="7" fill="1" visible="no" active="no"/>
-<layer number="23" name="tOrigins" color="15" fill="1" visible="no" active="no"/>
-<layer number="24" name="bOrigins" color="15" fill="1" visible="no" active="no"/>
-<layer number="25" name="tNames" color="7" fill="1" visible="no" active="no"/>
-<layer number="26" name="bNames" color="7" fill="1" visible="no" active="no"/>
-<layer number="27" name="tValues" color="7" fill="1" visible="no" active="no"/>
-<layer number="28" name="bValues" color="7" fill="1" visible="no" active="no"/>
+<layer number="1" name="Top" color="4" fill="1" visible="yes" active="no"/>
+<layer number="16" name="Bottom" color="1" fill="1" visible="yes" active="no"/>
+<layer number="17" name="Pads" color="2" fill="1" visible="yes" active="no"/>
+<layer number="18" name="Vias" color="2" fill="1" visible="yes" active="no"/>
+<layer number="19" name="Unrouted" color="6" fill="1" visible="yes" active="no"/>
+<layer number="20" name="Dimension" color="15" fill="1" visible="yes" active="no"/>
+<layer number="21" name="tPlace" color="7" fill="1" visible="yes" active="no"/>
+<layer number="22" name="bPlace" color="7" fill="1" visible="yes" active="no"/>
+<layer number="23" name="tOrigins" color="15" fill="1" visible="yes" active="no"/>
+<layer number="24" name="bOrigins" color="15" fill="1" visible="yes" active="no"/>
+<layer number="25" name="tNames" color="7" fill="1" visible="yes" active="no"/>
+<layer number="26" name="bNames" color="7" fill="1" visible="yes" active="no"/>
+<layer number="27" name="tValues" color="7" fill="1" visible="yes" active="no"/>
+<layer number="28" name="bValues" color="7" fill="1" visible="yes" active="no"/>
 <layer number="29" name="tStop" color="7" fill="3" visible="no" active="no"/>
 <layer number="30" name="bStop" color="7" fill="6" visible="no" active="no"/>
@@
 <layer number="35" name="tGlue" color="7" fill="4" visible="no" active="no"/>
 <layer number="36" name="bGlue" color="7" fill="5" visible="no" active="no"/>
-<layer number="37" name="tTest" color="7" fill="1" visible="no" active="no"/>
-<layer number="38" name="bTest" color="7" fill="1" visible="no" active="no"/>
+<layer number="37" name="tTest" color="7" fill="1" visible="yes" active="no"/>
+<layer number="38" name="bTest" color="7" fill="1" visible="yes" active="no"/>
 <layer number="39" name="tKeepout" color="4" fill="11" visible="no" active="no"/>
 <layer number="40" name="bKeepout" color="1" fill="11" visible="no" active="no"/>
@@
 <layer number="44" name="Drills" color="7" fill="1" visible="no" active="no"/>
 <layer number="45" name="Holes" color="7" fill="1" visible="no" active="no"/>
-<layer number="46" name="Milling" color="3" fill="1" visible="no" active="no"/>
-<layer number="47" name="Measures" color="7" fill="1" visible="no" active="no"/>
-<layer number="48" name="Document" color="7" fill="1" visible="no" active="no"/>
-<layer number="49" name="Reference" color="7" fill="1" visible="no" active="no"/>
-<layer number="50" name="dxf" color="7" fill="1" visible="no" active="no"/>
-<layer number="51" name="tDocu" color="6" fill="1" visible="no" active="no"/>
-<layer number="52" name="bDocu" color="7" fill="1" visible="no" active="no"/>
+<layer number="46" name="Milling" color="3" fill="1" visible="yes" active="no"/>
+<layer number="47" name="Measures" color="7" fill="1" visible="yes" active="no"/>
+<layer number="48" name="Document" color="7" fill="1" visible="yes" active="no"/>
+<layer number="49" name="Reference" color="7" fill="1" visible="yes" active="no"/>
+<layer number="50" name="dxf" color="7" fill="1" visible="yes" active="no"/>
+<layer number="51" name="tDocu" color="7" fill="1" visible="yes" active="no"/>
+<layer number="52" name="bDocu" color="7" fill="1" visible="yes" active="no"/>
 <layer number="90" name="Modules" color="5" fill="1" visible="yes" active="yes"/>
 <layer number="91" name="Nets" color="2" fill="1" visible="yes" active="yes"/>
@@
 <parts>
 <part name="R1" library="rcl" deviceset="R-US_" device="0207/7"/>
-<part name="R2" library="rcl" deviceset="R-US_" device="0207/7"/>
+<part name="R2" library="rcl" deviceset="R-US_" device="0207/5V"/>
 <part name="C1" library="rcl" deviceset="C-EU" device="025-025X050"/>
 <part name="C2" library="rcl" deviceset="C-EU" device="050-025X075"/>
@@
 <part name="R3" library="rcl" deviceset="R-US_" device="R0805" value="1M SMD"/>
 <part name="C3" library="rcl" deviceset="C-EU" device="C0805" value="100n SMD"/>
-<part name="LED1" library="led" deviceset="LED" device="5MM"/>
-<part name="LED2" library="led" deviceset="LED" device="5MM"/>
+<part name="LED1" library="led" deviceset="LED" device="3MM"/>
+<part name="LED2" library="led" deviceset="LED" device="3MM"/>
 <part name="Q1" library="gm-trans" deviceset="J201" device=""/>
 <part name="R4" library="rcl" deviceset="R-US_" device="0207/7"/>
@@
 <part name="P+5" library="supply1" deviceset="V+" device=""/>
 <part name="GND35" library="supply1" deviceset="GND" device=""/>
-<part name="JP8" library="pinhead" deviceset="PINHD-1X1" device=""/>
+<part name="JP_IN" library="pinhead" deviceset="PINHD-1X1" device=""/>
 <part name="JP9" library="pinhead" deviceset="PINHD-1X1" device=""/>
 <part name="GND36" library="supply1" deviceset="GND" device=""/>
-<part name="JP10" library="pinhead" deviceset="PINHD-1X1" device=""/>
+<part name="JP_OUT" library="pinhead" deviceset="PINHD-1X1" device=""/>
 <part name="JP11" library="pinhead" deviceset="PINHD-1X1" device=""/>
 <part name="GND37" library="supply1" deviceset="GND" device=""/>
@@
 <instance part="P+5" gate="1" x="58.42" y="99.06"/>
 <instance part="GND35" gate="1" x="5.08" y="35.56"/>
-<instance part="JP8" gate="G$1" x="-10.16" y="53.34" rot="R180"/>
+<instance part="JP_IN" gate="G$1" x="-10.16" y="53.34" rot="R180"/>
 <instance part="JP9" gate="G$1" x="-10.16" y="45.72" rot="R180"/>
 <instance part="GND36" gate="1" x="0" y="43.18"/>
-<instance part="JP10" gate="G$1" x="541.02" y="68.58"/>
+<instance part="JP_OUT" gate="G$1" x="541.02" y="68.58"/>
 <instance part="JP11" gate="G$1" x="541.02" y="60.96"/>
 <instance part="GND37" gate="1" x="530.86" y="58.42"/>
@@
 <wire x1="5.08" y1="53.34" x2="-7.62" y2="53.34" width="0.1524" layer="91"/>
 <junction x="5.08" y="53.34"/>
-<pinref part="JP8" gate="G$1" pin="1"/>
+<pinref part="JP_IN" gate="G$1" pin="1"/>
 </segment>
 </net>
@@
 <segment>
 <pinref part="POT_VOL" gate="G$1" pin="2"/>
-<pinref part="JP10" gate="G$1" pin="1"/>
+<pinref part="JP_OUT" gate="G$1" pin="1"/>
 <wire x1="538.48" y1="68.58" x2="528.32" y2="68.58" width="0.1524" layer="91"/>
 </segment>

Commit message: Ajustes no esquematico e no layout
Parts:
- removed C5, C6, C7: (no value), rcl:C-EU050-025X075
- removed JP6, JP7: (no value), pinhead:PINHD-1X1
- removed R10, R7, R8, R9: (no value), rcl:R-US_0207/7
- added SJ3, SJ4: (no value), jumper:SJ
Connections:
- removed net N$41: C22.1, C23.1, R38.1
- removed net N$7: C2.1, C5.2, R8.1
- removed net N$9: C6.1, C7.1, R10.1, R8.2
- new net TONE_IN: C22.1, C23.1, R38.1, SJ3.2
- new net TONE_OUT: POT_TONE/TREBLE.2, SJ4.1
- net GND: no longer C6.2, JP7.1, R7.2, R9.1
- net N$11: now also SJ4.2; no longer POT_TONE/TREBLE.2
- net N$6: now also C2.1, SJ3.1; no longer C7.2, JP6.1, R9.2
- net TONE/TREBLE_1: no longer R10.2
- net TONE/TREBLE_3: no longer C5.1, R7.1
Other:
- note added: "Azabache - Ligar resistor 47k em C24, capacitor 10n em R39, cap e chave scoop em POT_MIDS, jumper em C25"
- note added: "Fender/Marshall - montar jumper e deixar R39 em aberto"
- note removed: "AZABACHE SCOOP"
- note removed: "Fender - montar jumper e deixar R39 em aberto"
- moved on the sheet: C22, C23, C24, C25, POT_BASS, POT_MIDS, POT_TONE/TREBLE, R38, R39, SJ1

Commit message: Desenvolvimento do layout - roteamento da placa Pendente roteamento do terra e análises do esquematico e layout
Parts:
- removed JP12, JP13, JP14: (no value), pinhead:PINHD-1X1
- added C5: (no value), rcl:C-EU050-025X075
- added C6: (no value), rcl:CPOL-EUE2.5-6
- added C7: 100n SMD, rcl:C-EUC0805
- added JP+, JP-, JP6, JP7: (no value), pinhead:PINHD-1X1
- added Q8: J201, gm-trans:J201
- added R7: (no value), rcl:R-US_0207/5V
- added R8, R9: (no value), rcl:R-US_0207/7
- added SJ5: (no value), jumper:SJ
- R19: device rcl:R-US_0207/7 -> rcl:R-US_0207/5V
- renumbered JP4 to JP_BRT1, JP5 to JP_BRT2
Connections:
- removed net N$34: C20.2, POT_VOL.3, R36.2, R37.2
- new net N$14: C5.1, JP7.1
- new net N$7: C26.+, Q6.G, R40.1, R7.1
- new net N$9: C20.2, POT_VOL.3, R36.2, R37.2, R9.1, SJ5.2
- net GND: now also C3.2, C6.-, C7.2, JP-.1, JP6.1, R8.1; no longer JP12.1, JP13.1, JP14.1
- net N$10: now also C5.2, R9.2; no longer C26.+, Q6.G, R40.1
- net N$28: now also Q8.G
- net TONE_IN: now also Q8.S, R8.2
- net TONE_OUT: now also SJ5.1
- net V+: now also C3.1, C6.+, C7.1, JP+.1, Q8.D
- net VCC/2: now also R7.2
Other:
- note added: "Chave Bright/Gain"
- note added: "Ponto JP1 para chave Clean/Dirt Azabache"
- note added: "Pontos JP2 e JP3 apenas para chave Clean/Dirt no Azabache, se montado"
- note added: "Presence"
- note removed: "AZABACHE BRIGHT"
- moved on the sheet: C17, C18, C19, C20, C21, C3, JP11, JP2, JP3, JP_OUT, POT_VOL, Q5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

Commit message: Revisao do esquematico
Parts:
- added SJ6: (no value), jumper:SJ
Connections:
- net N$11: now also SJ6.2
- net N$6: now also SJ6.1
Other:
- moved on the sheet: C1, C2, C26, C4, JP9, JP_BRT1, JP_BRT2, JP_IN, LED1, LED2, Q1, Q6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

Commit message: Alteracoes e correcoes no esquematico e layout apos verificacao para montagem de Azabache/Spitfire/Dr Boogie
Parts:
- removed SJ6: (no value), jumper:SJ
- added C34, C38, C39, C40, C41, C42: (no value), rcl:C-EU025-025X050
- added C35, C36, C37: (no value), rcl:C-EU050-025X075
- added R10, R44, R47, R48: (no value), rcl:R-US_0207/7
- added R45: 1M SMD, rcl:R-US_R0805
- added R46: (no value), rcl:R-US_0207/5V
- C26: device rcl:CPOL-EUE2.5-6 -> rcl:C-EU025-025X050
- R11: device rcl:R-US_0207/7 -> rcl:R-US_R0805
Connections:
- removed net N$6: C2.1, SJ3.1, SJ6.1
- new net N$34: R4.1, R44.2
- new net N$38: C35.1, JP_IN.1, R45.2, R46.2
- new net N$39: C2.1, C36.2, R47.2, R48.2, SJ3.1
- net GND: now also C34.1, R10.2, R44.1, R45.1, R46.1, R47.1; no longer R4.1
- net N$11: now also C36.1, R48.1; no longer SJ6.2
- net N$13: no longer C33.1
- net N$16: now also C40.1
- net N$19: now also C41.2
- net N$2: now also C39.1
- net N$20: now also C41.1
- net N$22: now also C37.2
- net N$25: now also C42.2
- net N$26: now also C42.1
- net N$3: now also C33.1
- net N$4: now also C34.2, C39.2
- net N$42: now also C40.2
- net N$5: now also C35.2; no longer JP_IN.1
- net N$7: now also C26.2, C38.2; no longer C26.+
- net N$8: now also C26.1, C38.1; no longer C26.-
- net TONE/TREBLE_3: now also R10.1
- net V+: now also C37.1
Other:
- moved on the sheet: C1, C10, C14, C15, C16, C17, C18, C19, C20, C21, C22, C23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

Commit message: Ajustes no tonestack para contemplar montagens Fender/Marshall/Dumble
Parts:
- added SJ6: (no value), jumper:SJ
Connections:
- new net N$6: C25.1, POT_MIDS.2, SJ6.2
- net GND: no longer POT_MIDS.2
- net N$37: now also SJ6.1; no longer C25.1
Other:
- note added: "Fender - montar SJ1 e SJ6"
- note added: "Marshall - montar SJ1"
- note added: "Umble - montar R39 e deixar jumpers em aberto. Controle Mid ficará invertido em relação ao original."
- note removed: "Azabache - Ligar resistor 47k em C24, capacitor 10n em R39, cap e chave scoop em POT_MIDS, jumper em C25"
- note removed: "Fender/Marshall - montar jumper e deixar R39 em aberto"
- note removed: "Umble - montar R39 e deixar jumper em aberto"
- moved on the sheet: C25, POT_MIDS, R39, SJ1
