File: multipreamp-1.sch (EAGLE design)
At the start: 138 parts, among them Q1 J201, Q2 J201, Q3 J201, Q4 J201, Q5 J201, Q6 J201, Q7 J201, Q8 2N5088

Commit message: Ajustes no layout - troca de encapsulamento dos trimpots
Parts:
- R12, R27, R33, R39: device rcl:R-TRIMM64W -> rcl:R-TRIMM3296W
- R31: device rcl:R-US_0207/5V -> rcl:R-US_0207/7
Changed lines of the file:
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@@
 <grid distance="0.1" unitdist="inch" unit="inch" style="lines" multiple="1" display="no" altdistance="0.05" altunitdist="inch" altunit="inch"/>
 <layers>
-<layer number="1" name="Top" color="4" fill="1" visible="no" active="no"/>
-<layer number="16" name="Bottom" color="1" fill="1" visible="no" active="no"/>
-<layer number="17" name="Pads" color="2" fill="1" visible="no" active="no"/>
-<layer number="18" name="Vias" color="2" fill="1" visible="no" active="no"/>
-<layer number="19" name="Unrouted" color="6" fill="1" visible="no" active="no"/>
-<layer number="20" name="Dimension" color="15" fill="1" visible="no" active="no"/>
-<layer number="21" name="tPlace" color="7" fill="1" visible="no" active="no"/>
-<layer number="22" name="bPlace" color="7" fill="1" visible="no" active="no"/>
-<layer number="23" name="tOrigins" color="15" fill="1" visible="no" active="no"/>
-<layer number="24" name="bOrigins" color="15" fill="1" visible="no" active="no"/>
-<layer number="25" name="tNames" color="7" fill="1" visible="no" active="no"/>
-<layer number="26" name="bNames" color="7" fill="1" visible="no" active="no"/>
-<layer number="27" name="tValues" color="7" fill="1" visible="no" active="no"/>
-<layer number="28" name="bValues" color="7" fill="1" visible="no" active="no"/>
+<layer number="1" name="Top" color="4" fill="1" visible="yes" active="no"/>
+<layer number="16" name="Bottom" color="1" fill="1" visible="yes" active="no"/>
+<layer number="17" name="Pads" color="2" fill="1" visible="yes" active="no"/>
+<layer number="18" name="Vias" color="2" fill="1" visible="yes" active="no"/>
+<layer number="19" name="Unrouted" color="6" fill="1" visible="yes" active="no"/>
+<layer number="20" name="Dimension" color="15" fill="1" visible="yes" active="no"/>
+<layer number="21" name="tPlace" color="7" fill="1" visible="yes" active="no"/>
+<layer number="22" name="bPlace" color="7" fill="1" visible="yes" active="no"/>
+<layer number="23" name="tOrigins" color="15" fill="1" visible="yes" active="no"/>
+<layer number="24" name="bOrigins" color="15" fill="1" visible="yes" active="no"/>
+<layer number="25" name="tNames" color="7" fill="1" visible="yes" active="no"/>
+<layer number="26" name="bNames" color="7" fill="1" visible="yes" active="no"/>
+<layer number="27" name="tValues" color="7" fill="1" visible="yes" active="no"/>
+<layer number="28" name="bValues" color="7" fill="1" visible="yes" active="no"/>
 <layer number="29" name="tStop" color="7" fill="3" visible="no" active="no"/>
 <layer number="30" name="bStop" color="7" fill="6" visible="no" active="no"/>
@@
 <layer number="35" name="tGlue" color="7" fill="4" visible="no" active="no"/>
 <layer number="36" name="bGlue" color="7" fill="5" visible="no" active="no"/>
-<layer number="37" name="tTest" color="7" fill="1" visible="no" active="no"/>
-<layer number="38" name="bTest" color="7" fill="1" visible="no" active="no"/>
+<layer number="37" name="tTest" color="7" fill="1" visible="yes" active="no"/>
+<layer number="38" name="bTest" color="7" fill="1" visible="yes" active="no"/>
 <layer number="39" name="tKeepout" color="4" fill="11" visible="no" active="no"/>
 <layer number="40" name="bKeepout" color="1" fill="11" visible="no" active="no"/>
@@
 <layer number="44" name="Drills" color="7" fill="1" visible="no" active="no"/>
 <layer number="45" name="Holes" color="7" fill="1" visible="no" active="no"/>
-<layer number="46" name="Milling" color="3" fill="1" visible="no" active="no"/>
-<layer number="47" name="Measures" color="7" fill="1" visible="no" active="no"/>
-<layer number="48" name="Document" color="7" fill="1" visible="no" active="no"/>
-<layer number="49" name="Reference" color="7" fill="1" visible="no" active="no"/>
-<layer number="50" name="dxf" color="7" fill="1" visible="no" active="no"/>
-<layer number="51" name="tDocu" color="7" fill="1" visible="no" active="no"/>
-<layer number="52" name="bDocu" color="7" fill="1" visible="no" active="no"/>
+<layer number="46" name="Milling" color="3" fill="1" visible="yes" active="no"/>
+<layer number="47" name="Measures" color="7" fill="1" visible="yes" active="no"/>
+<layer number="48" name="Document" color="7" fill="1" visible="yes" active="no"/>
+<layer number="49" name="Reference" color="7" fill="1" visible="yes" active="no"/>
+<layer number="50" name="dxf" color="7" fill="1" visible="yes" active="no"/>
+<layer number="51" name="tDocu" color="7" fill="1" visible="yes" active="no"/>
+<layer number="52" name="bDocu" color="7" fill="1" visible="yes" active="no"/>
 <layer number="90" name="Modules" color="5" fill="1" visible="yes" active="yes"/>
 <layer number="91" name="Nets" color="2" fill="1" visible="yes" active="yes"/>
@@
 <part name="GND14" library="supply1" deviceset="GND" device=""/>
 <part name="GND15" library="supply1" deviceset="GND" device=""/>
-<part name="R12" library="rcl" deviceset="R-TRIMM" device="64W"/>
+<part name="R12" library="rcl" deviceset="R-TRIMM" device="3296W"/>
 <part name="POT_TREBLE/TONE" library="gm-pots" deviceset="POT" device="PCB"/>
 <part name="POT_GAIN" library="gm-pots" deviceset="POT" device="PCB"/>
@@
 <part name="GND26" library="supply1" deviceset="GND" device=""/>
 <part name="GND25" library="supply1" deviceset="GND" device=""/>
-<part name="R27" library="rcl" deviceset="R-TRIMM" device="64W"/>
+<part name="R27" library="rcl" deviceset="R-TRIMM" device="3296W"/>
 <part name="C27" library="rcl" deviceset="C-EU" device="050-025X075"/>
 <part name="JP7" library="pinhead" deviceset="PINHD-1X1" device=""/>
 <part name="R30" library="rcl" deviceset="R-US_" device="R0805" value="1M SMD"/>
-<part name="R31" library="rcl" deviceset="R-US_" device="0207/5V"/>
+<part name="R31" library="rcl" deviceset="R-US_" device="0207/7"/>
 <part name="R32" library="rcl" deviceset="R-US_" device="0207/7"/>
 <part name="D3" library="diode" deviceset="1N4148" device="DO35-7" value="1N4148"/>
@@
 <part name="R34" library="rcl" deviceset="R-US_" device="0207/7"/>
 <part name="R35" library="rcl" deviceset="R-US_" device="0207/7"/>
-<part name="R33" library="rcl" deviceset="R-TRIMM" device="64W"/>
+<part name="R33" library="rcl" deviceset="R-TRIMM" device="3296W"/>
 <part name="GND34" library="supply1" deviceset="GND" device=""/>
 <part name="C32" library="rcl" deviceset="C-EU" device="050-025X075"/>
@@
 <part name="R40" library="rcl" deviceset="R-US_" device="0207/7"/>
 <part name="R41" library="rcl" deviceset="R-US_" device="0207/7"/>
-<part name="R39" library="rcl" deviceset="R-TRIMM" device="64W"/>
+<part name="R39" library="rcl" deviceset="R-TRIMM" device="3296W"/>
 <part name="GND42" library="supply1" deviceset="GND" device=""/>
 <part name="JP8" library="pinhead" deviceset="PINHD-1X1" device=""/>

Commit message: Ajustes no esquematico e adicao de capacitores de bypass
Parts:
- added C44, C45: 100n SMD, rcl:C-EUC0805
Connections:
- removed net 9V_1: C1.+, C2.1, C29.1, Q7.D, Q8.C, R1.2, R2.1, R33.A, R39.A, R43.1
- removed net V+: C3.+, C4.1, Q1.D, Q3.D, R12.A, R2.2, R27.A, R3.1
- new net V+/1: C3.+, C4.1, C45.1, Q1.D, Q3.D, R12.A, R2.2, R27.A, R3.1
- new net V+/2: C1.+, C2.1, C29.1, C44.1, Q7.D, Q8.C, R1.2, R2.1, R33.A, R39.A, R43.1
- net GND: now also C44.2, C45.2
Other:
- moved on the sheet: C1, C2, C3, JP1, JP2, R1, R2, R25, R26

Commit message: Ajustes no layout e criacao do plano de terra DRC executado, sem erros
Other:
- moved on the sheet: C1, C2, C3, C4, C44, C45, C5, C6, JP1, JP2, R1, R2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

Commit message: Troca do potenciometro por modelo com layers corretos para silkagem na PCB Ajustes no layout
Parts:
- POT_BASS, POT_GAIN, POT_MIDS, POT_TREBLE/TONE, POT_VOL: device gm-pots:POTPCB -> PATSKO:POTPCB
